Commit message: UPDATE: add digital io

File: ethercat_motor_drive/description/ros2_control/motor_drive.ros2_control.xacro (robot description, xacro)
@@ -7,6 +7,7 @@
         <param name="master_id">0</param>
         <param name="control_frequency">100</param>
+        <!-- <plugin>mock_components/GenericSystem</plugin> -->
       </hardware>
-      <joint name="joint2">
+      <!-- <joint name="joint2">
         <state_interface name="position"/>
         <state_interface name="velocity"/>
@@ -24,5 +25,45 @@
           <param name="slave_config">$(find ethercat_motor_drive)/config/circulo.yaml</param>
         </ec_module>
-      </joint>
+      </joint> -->
+      <gpio name="beckhoff_input">
+        <state_interface name="d_1"/>
+        <state_interface name="d_2"/>
+        <state_interface name="d_3"/>
+        <state_interface name="d_4"/>
+        <state_interface name="d_5"/>
+        <state_interface name="d_6"/>
+        <state_interface name="d_7"/>
+        <state_interface name="d_8"/>
+        <ec_module name="EL1809">
+          <plugin>ethercat_generic_plugins/GenericEcSlave</plugin>
+          <param name="alias">0</param>
+          <param name="position">1</param>
+          <param name="slave_config">$(find ethercat_motor_drive)/config/el1809.yaml</param>
+        </ec_module>
+      </gpio>
+      <gpio name="beckhoff_output">
+        <command_interface name="d_1"/>
+        <command_interface name="d_2"/>
+        <command_interface name="d_3"/>
+        <command_interface name="d_4"/>
+        <command_interface name="d_5"/>
+        <command_interface name="d_6"/>
+        <command_interface name="d_7"/>
+        <command_interface name="d_8"/>
+        <command_interface name="d_9"/>
+        <command_interface name="d_10"/>
+        <command_interface name="d_11"/>
+        <command_interface name="d_12"/>
+        <command_interface name="d_13"/>
+        <command_interface name="d_14"/>
+        <command_interface name="d_15"/>
+        <command_interface name="d_16"/>
+        <ec_module name="EL2809">
+          <plugin>ethercat_generic_plugins/GenericEcSlave</plugin>
+          <param name="alias">0</param>
+          <param name="position">2</param>
+          <param name="slave_config">$(find ethercat_motor_drive)/config/el2809.yaml</param>
+        </ec_module>
+      </gpio>
     </ros2_control>
   </xacro:macro>
