Commit message: UPDATE: daily update

File: ethercat_motor_drive/description/config/motor_drive.config.xacro (robot description, xacro)
@@ -2,5 +2,7 @@
 <robot xmlns:xacro="http://www.ros.org/wiki/xacro" name="motor_drive">
   <link name="world"/>
+  <xacro:include filename="$(find ethercat_motor_drive)/description/urdf/robot_description.urdf.xacro" />
   <xacro:include filename="$(find ethercat_motor_drive)/description/ros2_control/motor_drive.ros2_control.xacro" />
+  <xacro:TechRobot/>
   <xacro:motor_drive/>
 </robot>

File: ethercat_motor_drive/description/ros2_control/motor_drive.ros2_control.xacro (robot description, xacro)
@@ -8,9 +8,10 @@
         <param name="control_frequency">100</param>
       </hardware>
-      <joint name="joint_1">
+      <joint name="joint2">
         <state_interface name="position"/>
         <state_interface name="velocity"/>
         <state_interface name="effort"/>
         <command_interface name="position"/>
+        <command_interface name="velocity"/>
         <command_interface name="reset_fault"/>
         <ec_module name="Maxon">
@@ -19,5 +20,5 @@
           <param name="position">0</param>
           <param name="mode_of_operation">8</param>
-          <param name="slave_config">$(find ethercat_motor_drive)/config/maxon_epos3_config.yaml</param>
+          <param name="slave_config">$(find ethercat_motor_drive)/config/stepper.yaml</param>
         </ec_module>
       </joint>

Commit message: UPDATE: add elfin

File: ethercat_motor_drive/description/config/motor_drive.config.xacro (robot description, xacro)
@@ -3,5 +3,6 @@
   <link name="world"/>
   <xacro:include filename="$(find ethercat_motor_drive)/description/urdf/robot_description.urdf.xacro" />
-  <xacro:include filename="$(find ethercat_motor_drive)/description/ros2_control/motor_drive.ros2_control.xacro" />
+  <xacro:include filename="$(find ethercat_motor_drive)/description/ros2_control/motor_drive_elfin.ros2_control.xacro" />
+  <!-- <xacro:include filename="$(find ethercat_motor_drive)/description/ros2_control/motor_drive.ros2_control.xacro" /> -->
   <!-- <xacro:include filename="$(find ethercat_motor_drive)/description/ros2_control/muti_motor_drive.ros2_control.xacro" /> -->
   <xacro:TechRobot/>

File: ethercat_motor_drive/description/ros2_control/motor_drive.ros2_control.xacro (robot description, xacro)
@@ -6,8 +6,8 @@
         <plugin>ethercat_driver/EthercatDriver</plugin>
         <param name="master_id">0</param>
-        <param name="control_frequency">100</param>
+        <param name="control_frequency">1000</param>
         <!-- <plugin>mock_components/GenericSystem</plugin> -->
       </hardware>
-      <!-- <joint name="joint2">
+      <joint name="joint2">
         <state_interface name="position"/>
         <state_interface name="velocity"/>
@@ -16,4 +16,5 @@
         <command_interface name="position"/>
         <command_interface name="velocity"/>
+        <command_interface name="effort"/>
         <command_interface name="reset_fault"/>
         <command_interface name="mode"/>
@@ -22,9 +23,9 @@
           <param name="alias">0</param>
           <param name="position">0</param>
-          <param name="mode_of_operation">8</param>
-          <param name="slave_config">$(find ethercat_motor_drive)/config/circulo.yaml</param>
+          <param name="mode_of_operation">9</param>
+          <param name="slave_config">$(find ethercat_motor_drive)/config/abb.yaml</param>
         </ec_module>
-      </joint> -->
-      <gpio name="beckhoff_input">
+      </joint>
+      <!-- <gpio name="beckhoff_input">
         <state_interface name="d_1"/>
         <state_interface name="d_2"/>
@@ -65,5 +66,5 @@
           <param name="slave_config">$(find ethercat_motor_drive)/config/el2809.yaml</param>
         </ec_module>
-      </gpio>
+      </gpio> -->
     </ros2_control>
   </xacro:macro>

File: ethercat_motor_drive/description/urdf/robot_description.urdf.xacro (robot description, xacro)
@@ -68,5 +68,5 @@
   </joint>
   <!-- joints - main serial chain -->
-  <joint name="joint0" type="fixed">
+  <joint name="joint0" type="revolute">
     <parent link="base_link"/>
     <child link="link0"/>
@@ -77,5 +77,5 @@
     <limit effort="1000.0" lower="-1" upper="1" velocity="2.5"/>
   </joint>
-  <joint name="joint1" type="fixed">
+  <joint name="joint1" type="revolute">
     <parent link="link0"/>
     <child link="link1"/>

Commit message: UPDATE: add MirroIO

File: ethercat_motor_drive/description/config/motor_drive.config.xacro (robot description, xacro)
@@ -3,7 +3,7 @@
   <link name="world"/>
   <xacro:include filename="$(find ethercat_motor_drive)/description/urdf/robot_description.urdf.xacro" />
-  <xacro:include filename="$(find ethercat_motor_drive)/description/ros2_control/io_elfin.ros2_control.xacro" />
+  <!-- <xacro:include filename="$(find ethercat_motor_drive)/description/ros2_control/io_elfin.ros2_control.xacro" /> -->
   <!-- <xacro:include filename="$(find ethercat_motor_drive)/description/ros2_control/motor_drive_elfin.ros2_control.xacro" /> -->
-  <!-- <xacro:include filename="$(find ethercat_motor_drive)/description/ros2_control/motor_drive.ros2_control.xacro" /> -->
+  <xacro:include filename="$(find ethercat_motor_drive)/description/ros2_control/motor_drive.ros2_control.xacro" />
   <!-- <xacro:include filename="$(find ethercat_motor_drive)/description/ros2_control/muti_motor_drive.ros2_control.xacro" /> -->
   <xacro:TechRobot/>

File: ethercat_motor_drive/description/ros2_control/motor_drive.ros2_control.xacro (robot description, xacro)
@@ -9,5 +9,5 @@
         <!-- <plugin>mock_components/GenericSystem</plugin> -->
       </hardware>
-      <joint name="joint2">
+      <!-- <joint name="joint2">
         <state_interface name="position"/>
         <state_interface name="velocity"/>
@@ -23,9 +23,9 @@
           <param name="alias">0</param>
           <param name="position">0</param>
-          <param name="mode_of_operation">9</param>
-          <param name="slave_config">$(find ethercat_motor_drive)/config/abb.yaml</param>
+          <param name="mode_of_operation">8</param>
+          <param name="slave_config">$(find ethercat_motor_drive)/config/leader56.yaml</param>
         </ec_module>
-      </joint>
-      <!-- <gpio name="beckhoff_input">
+      </joint> -->
+      <gpio name="beckhoff_input">
         <state_interface name="d_1"/>
         <state_interface name="d_2"/>
@@ -36,4 +36,12 @@
         <state_interface name="d_7"/>
         <state_interface name="d_8"/>
+        <state_interface name="d_9"/>
+        <state_interface name="d_10"/>
+        <state_interface name="d_11"/>
+        <state_interface name="d_12"/>
+        <state_interface name="d_13"/>
+        <state_interface name="d_14"/>
+        <state_interface name="d_15"/>
+        <state_interface name="d_16"/>
         <ec_module name="EL1809">
           <plugin>ethercat_generic_plugins/GenericEcSlave</plugin>
@@ -44,4 +52,20 @@
       </gpio>
       <gpio name="beckhoff_output">
+        <state_interface name="d_1"/>
+        <state_interface name="d_2"/>
+        <state_interface name="d_3"/>
+        <state_interface name="d_4"/>
+        <state_interface name="d_5"/>
+        <state_interface name="d_6"/>
+        <state_interface name="d_7"/>
+        <state_interface name="d_8"/>
+        <state_interface name="d_9"/>
+        <state_interface name="d_10"/>
+        <state_interface name="d_11"/>
+        <state_interface name="d_12"/>
+        <state_interface name="d_13"/>
+        <state_interface name="d_14"/>
+        <state_interface name="d_15"/>
+        <state_interface name="d_16"/>
         <command_interface name="d_1"/>
         <command_interface name="d_2"/>
@@ -61,10 +85,10 @@
         <command_interface name="d_16"/>
         <ec_module name="EL2809">
-          <plugin>ethercat_generic_plugins/GenericEcSlave</plugin>
+          <plugin>ethercat_generic_plugins/MirrorIO</plugin>
           <param name="alias">0</param>
           <param name="position">2</param>
           <param name="slave_config">$(find ethercat_motor_drive)/config/el2809.yaml</param>
         </ec_module>
-      </gpio> -->
+      </gpio>
     </ros2_control>
   </xacro:macro>
